File: pcb-hardware/keygame/keygame.kicad_pcb (KiCad board)
At the start: 2 copper layers, 56 x 84 mm, 45 parts, among them J1 DEBUG_HEADER, J2 POWER_HEADER, SW1 RIGHT, SW2 LEFT, SW3 B, SW4 A, SW5 DOWN, SW6 UP, U1 SeeeduinoXIAO, U2 SPI_OLED_SSH1106, U3 74HC165

Commit message: fixed J4
Parts:
- removed G***: LOGO, keygame:logo
- removed G***: LOGO, keygame:logo-big
- removed G***: LOGO, keygame:asteroids
- removed REF**: KiCAD Logo, Symbol:Symbol_KiCAD-Logo_CopperAndSilkScreenTop
- removed REF**: OSHW-Logo_5.7x6mm_SilkScreen, Symbol:OSHW-Logo_5.7x6mm_SilkScreen
- removed REF**: WEEE-Logo_5.6x8mm_SilkScreen, Symbol:WEEE-Logo_5.6x8mm_SilkScreen
- removed REF**: Symbol_CreativeCommons_SilkScreenTop_Type2_Big, Symbol:Symbol_CreativeCommons_SilkScreenTop_Type2_Big
- removed REF**: SIG, keygame:SIG
- added C10: 100nF, Capacitor_SMD:C_0402_1005Metric_Pad0.74x0.62mm_HandSolder, B.Cu at (171.7, 62.8)
- added C11: 1uF, Capacitor_SMD:C_0805_2012Metric_Pad1.18x1.45mm_HandSolder, B.Cu at (155.4, 63.8)
- added C12: 1uF, Capacitor_SMD:C_0805_2012Metric_Pad1.18x1.45mm_HandSolder, B.Cu at (154.9, 66.8)
- added C13: 100nF, Capacitor_SMD:C_0402_1005Metric_Pad0.74x0.62mm_HandSolder, B.Cu at (155.7, 62.2)
- added C14: 100nF, Capacitor_SMD:C_0402_1005Metric_Pad0.74x0.62mm_HandSolder, B.Cu at (171.7, 61.8)
- added C15: 100nF, Capacitor_SMD:C_0402_1005Metric_Pad0.74x0.62mm_HandSolder, B.Cu at (164.4, 54.5)
- added C16: 100nF, Capacitor_SMD:C_0402_1005Metric_Pad0.74x0.62mm_HandSolder, B.Cu at (160.9, 54.5)
- added C17: 100nF, Capacitor_SMD:C_0402_1005Metric_Pad0.74x0.62mm_HandSolder, B.Cu at (159.4, 69.2)
- added C18: 100nF, Capacitor_SMD:C_0402_1005Metric_Pad0.74x0.62mm_HandSolder, B.Cu at (158.4, 69.2)
- added C19: 100nF, Capacitor_SMD:C_0402_1005Metric_Pad0.74x0.62mm_HandSolder, B.Cu at (155.7, 65.2)
- added C20: 100nF, Capacitor_SMD:C_0402_1005Metric_Pad0.74x0.62mm_HandSolder, B.Cu at (164.4, 69.2)
- added C21: 10uF, Capacitor_SMD:C_1206_3216Metric_Pad1.33x1.80mm_HandSolder, B.Cu at (185.5, 48.2)
- added C22: 100nF, Capacitor_SMD:C_0402_1005Metric_Pad0.74x0.62mm_HandSolder, B.Cu at (152.3, 63.5)
- added C23: 10uF, Capacitor_SMD:C_1206_3216Metric_Pad1.33x1.80mm_HandSolder, B.Cu at (185.8, 37.2)
- added C8: 27pF, Capacitor_SMD:C_0402_1005Metric_Pad0.74x0.62mm_HandSolder, B.Cu at (175.0, 64.5)
- added C9: 100nF, Capacitor_SMD:C_0402_1005Metric_Pad0.74x0.62mm_HandSolder, B.Cu at (155.7, 61.2)
- added D1: RED, LED_SMD:LED_0402_1005Metric_Pad0.77x0.64mm_HandSolder, B.Cu at (175.1, 19.8)
- added D2: GRN, LED_SMD:LED_0402_1005Metric_Pad0.77x0.64mm_HandSolder, B.Cu at (176.1, 19.8)
- added D3: BLU, LED_SMD:LED_0402_1005Metric_Pad0.77x0.64mm_HandSolder, B.Cu at (175.6, 18.1)
- added F1: 500mA Hold, Fuse:Fuse_1206_3216Metric_Pad1.42x1.75mm_HandSolder, B.Cu at (174.3, 40.1)
- added J3: UART_HEADER, Connector_PinHeader_2.54mm:PinHeader_1x04_P2.54mm_Vertical, F.Cu at (140.5, 48.8)
- added J4: SWD_CONNECTOR, Connector_PinHeader_1.27mm:PinHeader_2x05_P1.27mm_Vertical_SMD, B.Cu at (184.9, 56.0)
- added JP1: JUMP_SCREEN_CS, Jumper:SolderJumper-3_P1.3mm_Bridged12_RoundedPad1.0x1.5mm, B.Cu at (169.1, 28.7)
- added P1: USB_C_CONNECTOR, Connector_USB:USB_C_Receptacle_HRO_TYPE-C-31-M-12, B.Cu at (186.2, 30.1)
- added R10: 1k, Resistor_SMD:R_0402_1005Metric_Pad0.72x0.64mm_HandSolder, B.Cu at (171.7, 60.8)
- added R11: 27, Resistor_SMD:R_0603_1608Metric_Pad0.98x0.95mm_HandSolder, B.Cu at (178.0, 32.2)
- added R12: 27, Resistor_SMD:R_0603_1608Metric_Pad0.98x0.95mm_HandSolder, B.Cu at (178.0, 33.8)
- added R13: 4.7k, Resistor_SMD:R_0402_1005Metric_Pad0.72x0.64mm_HandSolder, B.Cu at (171.7, 58.8)
- added R14: 300, Resistor_SMD:R_0402_1005Metric_Pad0.72x0.64mm_HandSolder, B.Cu at (174.0, 19.9)
- added R15: 4.7k, Resistor_SMD:R_0402_1005Metric_Pad0.72x0.64mm_HandSolder, B.Cu at (171.7, 59.8)
- added R16: 200, Resistor_SMD:R_0402_1005Metric_Pad0.72x0.64mm_HandSolder, B.Cu at (177.2, 19.9)
- added R17: 200, Resistor_SMD:R_0402_1005Metric_Pad0.72x0.64mm_HandSolder, B.Cu at (175.6, 17.1)
- added R18: 56k, Resistor_SMD:R_0402_1005Metric_Pad0.72x0.64mm_HandSolder, B.Cu at (179.0, 31.0)
- added R19: 10k, Resistor_SMD:R_0402_1005Metric_Pad0.72x0.64mm_HandSolder, B.Cu at (139.7, 63.2)
- added SW7: SW_SPST, Button_Switch_SMD:SW_SPST_PTS810, B.Cu at (135.5, 59.0)
- added SW9: SW_SPST, Button_Switch_SMD:SW_SPST_PTS810, B.Cu at (139.5, 59.0)
- added U4: NCP1117-3.3_SOT223, Package_TO_SOT_SMD:SOT-223-3_TabPin2, B.Cu at (183.5, 42.8)
- added Y1: 12MHz, Crystal:Crystal_HC52-8mm_Vertical, B.Cu at (175.0, 67.8)
- C1, C2, C3, C4, C5, C6: footprint Capacitor_SMD:C_0805_2012Metric_Pad1.15x1.40mm_HandSolder -> Capacitor_SMD:C_0402_1005Metric_Pad0.74x0.62mm_HandSolder; moved to B.Cu
- C7: value 100nF -> 27pF; footprint Capacitor_SMD:C_0805_2012Metric_Pad1.15x1.40mm_HandSolder -> Capacitor_SMD:C_0402_1005Metric_Pad0.74x0.62mm_HandSolder; moved to B.Cu
- R1: footprint Resistor_SMD:R_0805_2012Metric_Pad1.15x1.40mm_HandSolder -> Resistor_SMD:R_0805_2012Metric_Pad1.20x1.40mm_HandSolder; moved to B.Cu
- R2, R3, R4, R5, R6, R7, R9: footprint Resistor_SMD:R_0805_2012Metric_Pad1.15x1.40mm_HandSolder -> Resistor_SMD:R_0402_1005Metric_Pad0.72x0.64mm_HandSolder; moved to B.Cu
- R8: value 1k -> 10k; footprint Resistor_SMD:R_0805_2012Metric_Pad1.15x1.40mm_HandSolder -> Resistor_SMD:R_0402_1005Metric_Pad0.72x0.64mm_HandSolder; moved to B.Cu
- U1: value SeeeduinoXIAO -> RP2040; footprint keygame:Seeeduino XIAO-MOUDLE14P-2.54-21X17.8MM -> keygame:RP2040-QFN-56
- U3: value 74HC165 -> W25Q128JVS; footprint Package_DIP:DIP-16_W7.62mm_LongPads -> Package_SO:SOIC-8_5.23x5.23mm_P1.27mm; moved to B.Cu
- moved R8 30.4 mm to (134.5, 63.5), turned to 90 degrees
- moved U3 28.7 mm to (146.3, 61.5), turned to 0 degrees
- moved R9 27.5 mm to (140.7, 63.2), turned to 90 degrees
- moved U1 13.3 mm to (163.5, 62.0), turned to 270 degrees
- moved C7 8.65 mm to (171.2, 64.5), turned to 90 degrees
- moved R1 6.73 mm to (183.1, 67.7)
- moved R2 4.04 mm to (141.5, 72.8)
- moved SW6 3.54 mm to (144.5, 69.5)
- moved R6 3.48 mm to (186.0, 77.7)
- moved C4 3.35 mm to (141.5, 74.0)
- moved SW2 2.83 mm to (137.0, 77.0)
- moved R5 2.26 mm to (149.2, 80.2)
- moved SW1 2.24 mm to (152.0, 77.0)
- moved R3 1.90 mm to (141.8, 87.8)
- moved C1 1.75 mm to (141.8, 89.0)
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Connections:
- C1 pad 1: Net-(C1-Pad1) -> /BTN_DOWN
- C2 pad 1: Net-(C2-Pad1) -> /BTN_LEFT
- C3 pad 1: Net-(C3-Pad1) -> /BTN_RIGHT
- C4 pad 1: Net-(C4-Pad1) -> /BTN_UP
- C5 pad 1: Net-(C5-Pad1) -> /BTN_A
- C6 pad 1: Net-(C6-Pad1) -> /BTN_B
- C7 pad 1: +3V3 -> Net-(C7-Pad1)
- J1 pad 2: /MOSI -> /COPI
- J1 pad 6: /BUTTON_MISO -> /~USB_BOOT
- J1 pad 7: /BUTTON_CLK -> /RUN
- J1 pad 8: /BUTTON_LATCH -> GND
- R1 pad 1: Net-(R1-Pad1) -> /SPEAKER
- R2 pad 1: Net-(C4-Pad1) -> /BTN_UP
- R3 pad 1: Net-(C1-Pad1) -> /BTN_DOWN
- R4 pad 1: Net-(C2-Pad1) -> /BTN_LEFT
- R5 pad 1: Net-(C3-Pad1) -> /BTN_RIGHT
- R6 pad 1: Net-(C5-Pad1) -> /BTN_A
- R7 pad 1: Net-(C6-Pad1) -> /BTN_B
- R8 pad 1: Net-(R8-Pad1) -> +3V3
- R8 pad 2: GND -> /RUN
- R9 pad 1: Net-(R9-Pad1) -> /~QSPI_CS
- R9 pad 2: GND -> /~USB_BOOT
- SW1 pad 2: Net-(C3-Pad1) -> /BTN_RIGHT
- SW2 pad 2: Net-(C2-Pad1) -> /BTN_LEFT
- SW3 pad 2: Net-(C6-Pad1) -> /BTN_B
- SW4 pad 2: Net-(C5-Pad1) -> /BTN_A
- SW5 pad 2: Net-(C1-Pad1) -> /BTN_DOWN
- SW6 pad 2: Net-(C4-Pad1) -> /BTN_UP
- U1 pad 1: Net-(R1-Pad1) -> +3V3
- U1 pad 10: (no net) -> +3V3
- U1 pad 11: /MOSI -> Net-(U1-Pad11)
- U1 pad 12: +3V3 -> Net-(U1-Pad12)
- U1 pad 13: GND -> Net-(U1-Pad13)
- U1 pad 14: +5V -> Net-(U1-Pad14)
- U1 pad 15: +5V -> /SDA
- U1 pad 16: GND -> /SCL
- U1 pad 17: (no net) -> /BTN_A
- U1 pad 18: (no net) -> /BTN_B
- U1 pad 19: (no net) -> GND
- U1 pad 2: /SCREEN_DC -> /UART_TX
- U1 pad 20: GND -> Net-(C7-Pad1)
- U1 pad 3: /PADDLE -> /UART_RX
- U1 pad 4: /SCREEN_RST -> Net-(U1-Pad4)
- U1 pad 5: /BUTTON_MISO -> Net-(U1-Pad5)
- U1 pad 6: /BUTTON_CLK -> /CIPO
- U1 pad 7: /BUTTON_LATCH -> /SCREEN_CS_ALT
- U1 pad 8: /SCREEN_CS -> /SCK
- U1 pad 9: /SCK -> /COPI
- U2 pad 4: /MOSI -> /COPI
- U3 pad 1: /BUTTON_LATCH -> /~QSPI_CS
- U3 pad 2: /BUTTON_CLK -> /QSPI_D1
- U3 pad 3: Net-(C5-Pad1) -> /QSPI_D2
- U3 pad 4: Net-(C6-Pad1) -> GND
- U3 pad 5: (no net) -> /QSPI_D0
- U3 pad 6: (no net) -> /QSPI_CLK
- U3 pad 7: (no net) -> /QSPI_D3
- U3 pad 8: GND -> +3V3
Routing:
- net +3V3: track 213.5 -> 420.1 mm, vias 0 -> 16
- net /RUN: track 0.00 -> 135.2 mm, vias 0 -> 5
- net /GREEN_LED: track 0.00 -> 80.9 mm, vias 0 -> 4
- net /BLUE_LED: track 0.00 -> 78.4 mm, vias 0 -> 2
- net /BUTTON_MISO: track 77.3 -> 0.00 mm, vias 2 -> 0
- net /RED_LED: track 0.00 -> 73.5 mm, vias 0 -> 2
- net GND: track 3.23 -> 76.5 mm, vias 22 -> 37
- net /~USB_BOOT: track 0.00 -> 58.2 mm, vias 0 -> 1
- net Net-(C2-Pad1): track 48.2 -> 0.00 mm
- net Net-(C6-Pad1): track 47.3 -> 0.00 mm, vias 1 -> 0
- net /BUTTON_LATCH: track 47.2 -> 0.00 mm, vias 1 -> 0
- net /BTN_DOWN: track 0.00 -> 45.1 mm, vias 0 -> 1
- net /COPI: track 0.00 -> 44.0 mm, vias 0 -> 2
- net Net-(R12-Pad2): track 0.00 -> 43.9 mm, vias 0 -> 2
- net /BUTTON_CLK: track 43.8 -> 0.00 mm, vias 2 -> 0
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Other:
- net class Default: clearance 0.25 -> 0.2; trace_width 0.25 -> 0.2; via_dia 0.8 -> 0.5; via_drill 0.4 -> 0.3
- rule pad_to_mask_clearance: 0.051 -> 0
- rule trace_clearance: 0.25 -> 0.2
- rule trace_min: 0.25 -> 0.2
- board text added: "BOOT"
- board text added: "COPI"
- board text added: "IO"
- board text added: "MICRO"
- board text added: "RUN"
- board text added: "SCK"
- board text removed: "BUTTONS"
- board text removed: "LATCH"
- board text removed: "MISO"
- board text removed: "MOSI"
- board text removed: "Pinout A0: Speaker D1: Screen DC A2: Paddle D3: Screen Reset D4: Button MISO D5: Button CLK D6: Button Latch D7: Screen CS D8: Screen SCK D10: Screen MOSI"
- board text removed: "keygame Size 56mm X 84mm Corners 5mm radius Debug Header Pin 1 X=19.5mm, Y=79mm Power Header Pin 1 X=5mm, Y=69mm All M3 Mounting Holes 5mm X 5mm from corners"
