File: pcb-hardware/keygame/keygame.sch (KiCad schematic (older format))
At the start: 68 parts, among them J1 DEBUG_HEADER, J2 POWER_HEADER, SW1 RIGHT, SW2 LEFT, SW3 B, SW4 A, SW5 DOWN, SW6 UP, U2 SPI_OLED_SSH1106

Commit message: fixed J4
Parts:
- removed D?: LED_BGRA, symbol Device:LED_BGRA
- removed SW?: SW_DPST, symbol Switch:SW_DPST
- removed SW?: RESET, symbol Switch:SW_DPST
- added C21, C23: 10uF, Capacitor_SMD:C_1206_3216Metric_Pad1.33x1.80mm_HandSolder, symbol Device:C_Small
- added D1: RED, LED_SMD:LED_0402_1005Metric_Pad0.77x0.64mm_HandSolder, symbol Device:LED
- added D2: GRN, LED_SMD:LED_0402_1005Metric_Pad0.77x0.64mm_HandSolder, symbol Device:LED
- added D3: BLU, LED_SMD:LED_0402_1005Metric_Pad0.77x0.64mm_HandSolder, symbol Device:LED
- added F1: 500mA Hold, Fuse:Fuse_1206_3216Metric_Pad1.42x1.75mm_HandSolder, symbol Device:Polyfuse_Small
- added J3: UART_HEADER, Connector_PinHeader_2.54mm:PinHeader_1x04_P2.54mm_Vertical, symbol Connector_Generic:Conn_01x04
- added SW7, SW9: SW_SPST, Button_Switch_SMD:SW_SPST_PTS810, symbol Switch:SW_SPST
- added U4: NCP1117-3.3_SOT223, Package_TO_SOT_SMD:SOT-223-3_TabPin2, symbol Regulator_Linear:NCP1117-3.3_SOT223
- C1, C2, C3, C4, C5, C6: footprint Capacitor_SMD:C_0805_2012Metric_Pad1.15x1.40mm_HandSolder -> Capacitor_SMD:C_0402_1005Metric_Pad0.74x0.62mm_HandSolder
- C10, C13, C14, C15, C16, C17, C18, C19, C20, C22, C7, C8, C9: renamed from C?; footprint (none) -> Capacitor_SMD:C_0402_1005Metric_Pad0.74x0.62mm_HandSolder
- C11, C12: renamed from C?; footprint (none) -> Capacitor_SMD:C_0805_2012Metric_Pad1.18x1.45mm_HandSolder
- J4: renamed from J?; value Conn_ARM_JTAG_SWD_10 -> SWD_CONNECTOR; footprint (none) -> Connector_PinHeader_1.27mm:PinHeader_2x05_P1.27mm_Vertical_SMD
- JP1: renamed from JP?; footprint (none) -> Jumper:SolderJumper-3_P1.3mm_Bridged12_RoundedPad1.0x1.5mm
- P1: renamed from P?; value USB_C_Plug -> USB_C_CONNECTOR; footprint (none) -> Connector_USB:USB_C_Receptacle_HRO_TYPE-C-31-M-12
- R1: footprint Resistor_SMD:R_0805_2012Metric_Pad1.15x1.40mm_HandSolder -> Resistor_SMD:R_0805_2012Metric_Pad1.20x1.40mm_HandSolder
- R10, R13, R14, R15, R16, R17, R18, R19, R8, R9: renamed from R?; footprint (none) -> Resistor_SMD:R_0402_1005Metric_Pad0.72x0.64mm_HandSolder
- R11, R12: renamed from R?; footprint (none) -> Resistor_SMD:R_0603_1608Metric_Pad0.98x0.95mm_HandSolder
- R2, R3, R4, R5, R6, R7: footprint Resistor_SMD:R_0805_2012Metric_Pad1.15x1.40mm_HandSolder -> Resistor_SMD:R_0402_1005Metric_Pad0.72x0.64mm_HandSolder
- U1: renamed from U?; footprint RP2040_minimal:RP2040-QFN-56 -> keygame:RP2040-QFN-56
- Y1: renamed from Y?; footprint (none) -> Crystal:Crystal_HC52-8mm_Vertical
- gave numbers to parts that had none: 1
Connections:
- net MOSI is gone; now on net COPI: J1.2 (Pin_2)
- net +1V1: now also C10.1, C11.1, C9.1; no longer C10.2, C11.2, C9.2
- net +3V3: now also C12.1, C13.1, C14.1, C15.1, C16.1, C17.1, C18.1, C19.1, C20.1, C23.1, D1.2 (A), D2.2 (A), D3.2 (A), J3.1 (Pin_1), U4.2 (VO); no longer C12.2, C13.2, C14.2, C15.2, C16.2, C17.2, C18.2, C19.2, C20.2
- net +5V: now also F1.2
- net GND: now also C10.2, C11.2, C12.2, C13.2, C14.2, C15.2, C16.2, C17.2, C18.2, C19.2, C20.2, C9.2, J1.8 (Pin_8), C21.2, C23.2, J3.4 (Pin_4), SW7.1 (A), SW9.1 (A), U4.1 (GND); no longer C10.1, C11.1, C12.1, C13.1, C14.1, C15.1, C16.1, C17.1, C18.1, C19.1, C20.1, C9.1
- net RUN: now also J1.7 (Pin_7), SW7.2 (B)
- net UART_RX: now also J3.3 (Pin_3)
- net UART_TX: now also J3.2 (Pin_2)
- net ~USB_BOOT: now also J1.6 (Pin_6), SW9.2 (B)
- net at R14.1: now also D1.1 (K)
- net at R16.1: now also D2.1 (K)
- net at R17.1: now also D3.1 (K)
- new net: C21.1, F1.1, U4.3 (VI)
- no-connect marks 2 -> 22
Other:
- note added: "128Mb\nFlash Mem"
- note added: "3.3V Regulator"
- note added: "Connectors"
- note added: "RP2040\nMain Micro"
- note removed: "Expansion\nPorts"
- note removed: "Inputs (Buttons, Paddle)"
- moved on the sheet: C1, C10, C11, C12, C13, C14, C15, C16, C17, C18, C19, C2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
